File: hardware/boards/main-control-board/main-control-board-esp32.kicad_sch (KiCad schematic)
At the start: 3 parts, among them J7 Conn_ESP32, J8 Conn_ESP32

Commit message: feat(pcb): main control board rev3 (#66, #62)
* add extension port

* update BOM

* update expected nets

* update README.md for main control board: clarify extension port details and specify strapping pins and UART connections

* update silkscreen layer for main control board: add knockout effect to VCC and voltage labels

* add ESP antenna keepout

* add 100nF to U4 dVdt

* add capacitor next to pin 28 of PCA

* update hardware documentation: clarify power distribution and GPIO pin usage on the main control board, including details on USB-C connections and extension headers

* update silkscreen text on main control board: change label from "GP9" to "BOOT" and modify "GP8" to "GP8*"

* docs(pcb): add main control board revision 3 preview image
Parts:
- added C7: 100nF, Capacitor_SMD:C_0603_1608Metric, symbol Device:C
Connections:
- net +3.3V: now also C7.1
- net GND: now also C7.2
- net GP7: now reaches ESP2.11 (GP7), J8.2 (Pin_2)
- net GP8: now reaches ESP2.12 (GP8), J8.3 (Pin_3)
- net GP9: now reaches ESP2.13 (GP9), J8.4 (Pin_4)
- net GP10: now reaches ESP2.14 (GP10), J8.5 (Pin_5)
- net GP20: now reaches ESP2.17 (RX), J8.8 (Pin_8)
- net GP21: now reaches ESP2.18 (TX), J8.9 (Pin_9)
