File: hardware/boards/main-control-board/main-control-board.kicad_pcb (KiCad board)
At the start: 2 copper layers, 80.5 x 50 mm, 40 parts, among them J1 Conn_01x02_Pin_Speaker, J2 Conn_OLED, J3 Conn_extension, J4 Conn_extension_2, J7 Conn_ESP32, J8 Conn_ESP32, U1 PCA9685PW,118, U2 HX PZ2.54-3X5P ZZ, U3 MAX98357AETE+T, U4 TPS259571DSGR

Commit message: feat(pcb): main control board rev3 (#66, #62)
* add extension port

* update BOM

* update expected nets

* update README.md for main control board: clarify extension port details and specify strapping pins and UART connections

* update silkscreen layer for main control board: add knockout effect to VCC and voltage labels

* add ESP antenna keepout

* add 100nF to U4 dVdt

* add capacitor next to pin 28 of PCA

* update hardware documentation: clarify power distribution and GPIO pin usage on the main control board, including details on USB-C connections and extension headers

* update silkscreen text on main control board: change label from "GP9" to "BOOT" and modify "GP8" to "GP8*"

* docs(pcb): add main control board revision 3 preview image
Parts:
- added C6: 100nF, Capacitor_SMD:C_0603_1608Metric, F.Cu at (188.8, 92.5)
- added C7: 100nF, Capacitor_SMD:C_0603_1608Metric, F.Cu at (174.1, 93.1)
- J4: value Conn_extension_2 -> Conn_02x06_Odd_Even; footprint Connector_PinHeader_2.54mm:PinHeader_1x04_P2.54mm_Vertical -> Connector_PinHeader_2.54mm:PinHeader_2x06_P2.54mm_Vertical
- moved C1 39.6 mm to (145.3, 113.1), turned to 90 degrees
- moved R13 13.5 mm to (126.3, 116.0)
- moved D2 13.4 mm to (128.7, 116.0)
- moved C3 12.1 mm to (118.0, 93.8)
- moved C2 11.9 mm to (151.7, 92.8)
- moved NT1 11.7 mm to (146.2, 89.3)
- moved R12 11.0 mm to (122.0, 94.7)
- moved TP1 10.5 mm to (114.0, 107.1)
- moved TP2 10.4 mm to (114.0, 103.8)
- moved R5 10.1 mm to (147.1, 113.2)
- moved U1 10.0 mm to (138.6, 108.1)
- moved U2 10.0 mm to (138.2, 90.5)
- moved J1 10.0 mm to (116.4, 114.4)
- moved R3 10.0 mm to (139.6, 116.1)
- moved R4 10.0 mm to (142.1, 116.1)
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Connections:
- net Net-(J8-Pin_5) renamed /ESP32/GP10
- J4 pad 2: +3.3V -> /ESP32/GP21
- J4 pad 4: /ESP32/GP6 -> /ESP32/GP20
- J8 pad 2: Net-(J8-Pin_2) -> /ESP32/GP7
- J8 pad 3: Net-(J8-Pin_3) -> /ESP32/GP8
- J8 pad 4: Net-(J8-Pin_4) -> /ESP32/GP9
- J8 pad 8: Net-(J8-Pin_8) -> /ESP32/GP20
- J8 pad 9: Net-(J8-Pin_9) -> /ESP32/GP21
- U4 pad 1: unconnected-(U4-dVdt-Pad1) -> Net-(U4-dVdt)
Routing:
- net +3.3V: track 126.8 -> 167.2 mm
- net /I2S_BCLK: track 72.5 -> 96.9 mm, vias 2 -> 3
- net /ESP32/GP9: track 0.00 -> 24.3 mm
- net /ESP32/GP8: track 0.00 -> 20.3 mm
- net /I2S_LRC: track 74.3 -> 94.6 mm, vias 2 -> 3
- net /ESP32/GP7: track 0.00 -> 17.3 mm
- net /ESP32/GP20: track 0.00 -> 16.4 mm
- net /ESP32/GP21: track 0.00 -> 14.7 mm
- net /ESP32/GP5: track 52.8 -> 64.7 mm
- net /I2C_SCL: track 78.2 -> 89.9 mm
- net /I2C_SDA: track 82.6 -> 93.9 mm
- net /PCA/SERVO_5V: track 48.6 -> 59.3 mm
- net /I2S_DIN: track 74.6 -> 85.0 mm
- net GND: track 21.0 -> 11.6 mm, vias 38 -> 45
- net Net-(U4-dVdt): track 0.00 -> 3.09 mm
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- added copper zone on F.Cu, net /Audio/AUDIO_5V
Other:
- board size 80.5 x 50 mm -> 90.5 x 50 mm
- board text added: "BCLK"
- board text added: "BOOT"
- board text added: "GP20"
- board text added: "GP21"
- board text added: "GP8*"
- board text added: "I2S"
- board text added: "LRC"
- board text added: "TINY SOFTWARE ENGINEER Main Control Board HW REV #3 | 2026-10-06 github.com/jamro/tiny-engineer"
- board text removed: "TINY SOFTWARE ENGINEER Main Control Board HW REV #2 | 2026-09-24 github.com/jamro/tiny-engineer"

Commit message: feat(pcb): update main control board design with new silkscreen graphics and layout adjustments
* Added new graphics to the silkscreen layer, including "SCAN TO ASSEMBLE" and "HUMAN, I NEED A BODY!" texts.
* Updated the PCB design to include a QR code linking to the project website.
* Rearranged designators in the kicad_pro file for better organization.
Routing:
- net GND: vias 45 -> 44
Other:
- board text added: "HUMAN, I NEED A BODY!"
- board text added: "SCAN TO ASSEMBLE. PLEASE?"
- board text added: "TINY SOFTWARE ENGINEER Main Control Board HW REV #3 | 2026-10-06 https://tinyengineer.dev"
- board text removed: "TINY SOFTWARE ENGINEER Main Control Board HW REV #3 | 2026-10-06 github.com/jamro/tiny-engineer"
Changed lines of the file:
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@@
+	)
+	(gr_line
+		(start 130 103.5)
+		(end 130 102.5)
+		(stroke
+			(width 0.1)
+			(type default)
+		)
+		(layer "B.SilkS")
+	)
+	(gr_line
+		(start 130 103.5)
+		(end 160 103.5)
+		(stroke
+			(width 0.1)
+			(type default)
+		)
+		(layer "B.SilkS")
+	)
+	(gr_line
+		(start 160 103.5)
+		(end 160 90)
+		(stroke
+			(width 0.1)
+			(type default)
+		)
+		(layer "B.SilkS")
 	)
 	(gr_line
@@
 		(layer "Edge.Cuts")
 	)
-	(gr_text "TINY SOFTWARE ENGINEER\nMain Control Board\nHW REV #3 | 2026-10-06\ngithub.com/jamro/tiny-engineer"
+	(gr_text "TINY SOFTWARE ENGINEER\nMain Control Board\nHW REV #3 | 2026-10-06\nhttps://tinyengineer.dev"
 		(at 151.4 114 0)
 		(layer "F.SilkS")
@@
 		)
 	)
+	(gr_text "SCAN TO ASSEMBLE.\nPLEASE?"
+		(at 145.5 101 0)
+		(layer "B.SilkS")
+		(effects
+			(font
+				(size 0.8 0.8)
+				(thickness 0.12)
+			)
+			(justify left mirror)
+		)
+	)
 	(gr_text "DO NOT USE ESP USB WHILE BOARD USB IS CONNECTED!"
 		(at 179.705 86.6 0)
@@
 		)
 	)
+	(gr_text "HUMAN, I NEED A BODY!"
+		(at 145.5 98.5 0)
+		(layer "B.SilkS")
+		(effects
+			(font
+				(size 0.8 0.8)
+				(thickness 0.16)
+				(bold yes)
+			)
+			(justify left mirror)
+		)
+	)
 	(gr_text "SPEAKER"
 		(at 116 103.6 0)
@@
 			(justify mirror)
 		)
+	)
+	(barcode
+		(at 152.908 96.266 0)
+		(layer "B.SilkS")
+		(size 12 12)
+		(text "https://tinyengineer.dev/q/pcb-rev3")
+		(text_height 1)
+		(type qr)
+		(ecc_level M)
+		(hide yes)
+		(knockout no)
 	)
 	(segment
@@
 	)
 	(via
-		(at 158.115 90.805)
+		(at 157.734 88.9)
 		(size 0.8)
 		(drill 0.4)
@@
 	)
 	(via
-		(at 158.115 89.535)
+		(at 158.877 88.9)
 		(size 0.8)
 		(drill 0.4)
@@
 	)
 	(via
-		(at 158.115 92.075)
-		(size 0.8)
-		(drill 0.4)
-		(layers "F.Cu" "B.Cu")
-		(free yes)
-		(net "GND")
-	)
-	(via
-		(at 159.168235 104.2)
-		(size 0.8)
-		(drill 0.4)
-		(layers "F.Cu" "B.Cu")
-		(free yes)
-		(net "GND")
-	)
-	(via
-		(at 149.168235 104.2)
-		(size 0.8)
-		(drill 0.4)
-		(layers "F.Cu" "B.Cu")
-		(free yes)
-		(net "GND")
-	)
-	(via
-		(at 147.168235 104.2)
+		(at 159.168235 104.5)
+		(size 0.8)
+		(drill 0.4)
+		(layers "F.Cu" "B.Cu")
+		(free yes)
+		(net "GND")
+	)
+	(via
+		(at 149.168235 104.5)
+		(size 0.8)
+		(drill 0.4)
+		(layers "F.Cu" "B.Cu")
+		(free yes)
+		(net "GND")
+	)
+	(via
+		(at 147.168235 104.5)
 		(size 0.8)
 		(drill 0.4)
@@
 	)
 	(via
-		(at 158.168235 104.2)
+		(at 158.168235 104.5)
 		(size 0.8)
 		(drill 0.4)
@@
 	)
 	(via
-		(at 157.168235 104.2)
-		(size 0.8)
-		(drill 0.4)
-		(layers "F.Cu" "B.Cu")
-		(free yes)
-		(net "GND")
-	)
-	(via
-		(at 148.168235 104.2)
-		(size 0.8)
-		(drill 0.4)
+		(at 157.168235 104.5)
+		(size 0.8)
+		(drill 0.4)
+		(layers "F.Cu" "B.Cu")
+		(free yes)
+		(net "GND")
+	)
+	(via
+		(at 148.168235 104.5)
+		(size 0.8)
+		(drill 0.4)
